Commit message: mapping code added

File: packages/sentry/sentry_urdf/urdf/sentry.xacro (robot description, xacro)
@@ -8,8 +8,6 @@
     <xacro:property name="bodyheight" value="0.5" />
     <xacro:property name="bodyclearance" value="0.4" />  <!--clearance from bottom of box to ground-->
-    <!-- placement of main body relative to base link frame -->
-    <xacro:property name="bodyOX" value="${-half_bodylen}" />
-    <xacro:property name="bodyOY" value="0" />
-    <xacro:property name="bodyOZ" value="0.45" />
+    <!-- how far the center of the robot should be above the ground -->
+    <xacro:property name="zDisp" value="0.6" />
     <xacro:property name="mastlen" value="${bodywidth/10}" />
     <xacro:property name="mastwidth" value="${bodywidth}" />
@@ -65,8 +63,5 @@
             <parent link="base_link"/>
             <child link="${prefix}_wheel"/>
-            <!--
-            <origin xyz="0 ${left*track/2} ${tirerad}" rpy="0 ${M_PI/2} ${M_PI/2}"/>
-            -->
-            <origin xyz="${displacement} ${left*track/2} ${-bodyheight/2}" rpy="0 ${M_PI/2} ${M_PI/2}"/>
+            <origin xyz="${displacement} ${left*track/2} ${-bodyheight/2 + zDisp}" rpy="0 ${M_PI/2} ${M_PI/2}"/>
             <limit effort="100" velocity="15" />
             <joint_properties damping="0.0" friction="0.0" />
@@ -97,5 +92,5 @@
             <parent link="base_link"/>
             <child link="${prefix}_big_wheel"/>
-            <origin xyz="${displacement} ${left*track/2} ${bigtirerad}" rpy="0 ${M_PI/2} ${M_PI/2}"/>
+            <origin xyz="${displacement} ${left*track/2} ${bigtirerad + zDisp}" rpy="0 ${M_PI/2} ${M_PI/2}"/>
             <limit effort="100" velocity="15" />
             <joint_properties damping="0.0" friction="0.0" />
@@ -115,5 +110,5 @@
         <inertial>
             <!--assign almost all the mass to the main body box; set m= 100kg; treat I as approx m*r^2 -->
-            <mass value="2" />
+            <mass value="100" />
             <inertia ixx="10" ixy="0" ixz="0"
               iyy="10" iyz="0"
@@ -124,5 +119,5 @@
         <parent link="base_link"/>
         <child link="mast"/>
-        <origin xyz="${bodylen/4} 0 ${mastheight/2 + bodyheight/2}" rpy="0 0 0"/>
+        <origin xyz="${bodylen/4} 0 ${mastheight/2 + bodyheight/2 + zDisp}" rpy="0 0 0"/>
     </joint>
     <link name="base_link">
@@ -131,8 +126,5 @@
                 <box size="${bodylen} ${bodywidth} ${bodyheight}"/>
             </geometry>
-            <!--
-            <origin xyz="${bodyOX} ${bodyOY} ${bodyOZ}" rpy="0 0 0"/>
-            -->
-            <origin xyz="0 0 0" rpy="0 0 0"/>
+            <origin xyz="0 0 ${zDisp}" rpy="0 0 0"/>
         </visual>
         <collision>
@@ -140,8 +132,5 @@
                 <box size="${bodylen} ${bodywidth} ${bodyheight}"/>
             </geometry>
-            <!--
-            <origin xyz="${bodyOX} ${bodyOY} ${bodyOZ}" rpy="0 0 0"/>
-            -->
-            <origin xyz="0 0 0" rpy="0 0 0"/>
+            <origin xyz="0 0 ${zDisp}" rpy="0 0 0"/>
         </collision>
         <inertial>
@@ -156,5 +145,4 @@
   <link name="lidar_link">
       <collision>
-          <origin xyz="0 0 0" rpy="0 0 0"/>
           <geometry>
               <!-- coarse LIDAR model; a simple box -->
@@ -163,5 +151,4 @@
       </collision>
       <visual>
-          <origin xyz="0 0 0" rpy="0 0 0" />
           <geometry>
               <box size="${lidar_cube_size} ${lidar_cube_size} ${lidar_cube_size}" />
@@ -173,5 +160,4 @@
       <inertial>
           <mass value="4.0" />
-          <origin xyz="0 0 0" rpy="0 0 0"/>
           <inertia ixx="0.01" ixy="0" ixz="0" iyy="0.01" iyz="0" izz="0.01" />
       </inertial>
@@ -180,5 +166,5 @@
   <joint name="lidar_joint" type="fixed">
       <axis xyz="0 1 0" />
-      <origin xyz="${bodylen/2 + lidar_cube_size/2} 0 ${lidar_cube_size/2 - bodyheight/2}" rpy="0 0 0"/>
+      <origin xyz="${bodylen/2 + lidar_cube_size/2} 0 ${lidar_cube_size/2 - bodyheight/2 + zDisp}" rpy="0 0 0"/>
       <parent link="base_link"/>
       <child link="lidar_link"/>
@@ -188,5 +174,5 @@
     <sensor type="gpu_ray" name="sick_lidar_sensor">
       <pose>0 0 0 0 0 0</pose>
-      <visualize>false</visualize>
+      <visualize>true</visualize>
       <update_rate>40</update_rate>
       <ray>
@@ -232,23 +218,4 @@
     <xacro:big_wheel prefix="left" left="1" displacement="${-(bodylen/2 - 1.25*bigtirerad)}"/>
     <xacro:big_wheel prefix="right" left="-1" displacement="${-(bodylen/2 - 1.25*bigtirerad)}"/>
-<!--
-    <xacro:macro name="wheel_controller_plugin" params="wheelnum">
-        <plugin name="${wheelnum}_wheel_controller" filename="libgazebo_ros_diff_drive.so">
-            <alwaysOn>true</alwaysOn>
-            <updateRate>100</updateRate>
-            <leftJoint>right${wheelnum}_wheel_joint</leftJoint>
-            <rightJoint>left${wheelnum}_wheel_joint</rightJoint>
-            <wheelSeparation>${track}</wheelSeparation>
-            <wheelDiameter>${tirediam}</wheelDiameter>
-            <torque>200</torque>
-            <commandTopic>cmd_vel</commandTopic>
-            <odometryTopic>odom</odometryTopic>
-            <odometryFrame>odom</odometryFrame>
-            <robotBaseFrame>base_link</robotBaseFrame>
-            <publishWheelTF>true</publishWheelTF>
-            <publishWheelJointState>true</publishWheelJointState>
-        </plugin>
-    </xacro:macro>
- -->
     <xacro:macro name="wheel_controller_plugin" params="wheelset1 wheelset2">
       <plugin name="${wheelset1}_${wheelset2}_skid_steer_drive_controller" filename="libgazebo_ros_skid_steer_drive.so">
@@ -264,4 +231,10 @@
         <torque>200</torque>
         <topicName>cmd_vel</topicName>
+        <commandTopic>cmd_vel</commandTopic>
+        <odometryTopic>odom</odometryTopic>
+        <odometryFrame>odom</odometryFrame>
+        <broadcastTF>1</broadcastTF>
+        <publishWheelTF>true</publishWheelTF>
+        <publishWheelJointState>true</publishWheelJointState>
       </plugin>
     </xacro:macro>
@@ -271,28 +244,4 @@
         <xacro:wheel_controller_plugin wheelset1="3" wheelset2="1"/>
         <xacro:wheel_controller_plugin wheelset1="2" wheelset2="2"/>
-        <!--
-        <xacro:wheel_controller_plugin wheelnum="0" />
-        <xacro:wheel_controller_plugin wheelnum="1" />
-        <xacro:wheel_controller_plugin wheelnum="2" />
-        <xacro:wheel_controller_plugin wheelnum="3" />
-        <xacro:wheel_controller_plugin wheelnum="4" />
-         -->
-<!--
-        <plugin name="big_wheel_controller" filename="libgazebo_ros_diff_drive.so">
-            <alwaysOn>true</alwaysOn>
-            <updateRate>100</updateRate>
-            <leftJoint>left_big_wheel_joint</leftJoint>
-            <rightJoint>right_big_wheel_joint</rightJoint>
-            <wheelSeparation>${track}</wheelSeparation>
-            <wheelDiameter>${bigtirediam}</wheelDiameter>
-            <torque>200</torque>
-            <commandTopic>cmd_vel</commandTopic>
-            <odometryTopic>odom</odometryTopic>
-            <odometryFrame>odom</odometryFrame>
-            <robotBaseFrame>base_link</robotBaseFrame>
-            <publishWheelTF>true</publishWheelTF>
-            <publishWheelJointState>true</publishWheelJointState>
-        </plugin>
- -->
     </gazebo>
     <xacro:macro name="friction_macro" params="wheelnum constant">

Commit message: point click interface working like a baws

File: packages/sentry/sentry_urdf/urdf/sentry.xacro (robot description, xacro)
@@ -10,4 +10,5 @@
     <!-- how far the center of the robot should be above the ground -->
     <xacro:property name="zDisp" value="0.6" />
+    <xacro:property name="default_mass" value="1.0" />
     <xacro:property name="mastlen" value="${bodywidth/10}" />
     <xacro:property name="mastwidth" value="${bodywidth}" />
@@ -27,14 +28,4 @@
     <xacro:property name="wheelspacing" value="${(bodylen - 4*tirediam - tinywheelspacing)/3}" />
     <xacro:property name="M_PI" value="3.1415926535897931" />
-    <!--here is a default inertia matrix with small, but legal values; use this when don't need accuracy for I -->
-    <!--model will assign inertia matrix dominated by main body box -->
-    <xacro:macro name="default_inertial" params="mass">
-        <inertial>
-            <mass value="${mass}" />
-            <inertia ixx="0.01" ixy="0.0" ixz="0.0"
-         iyy="0.01" iyz="0.0"
-         izz="0.01" />
-        </inertial>
-    </xacro:macro>
     <!-- left = 1 if its the left wheel -1 if its the right wheel. displacement says how back/forward
     the wheel is from the center-->
@@ -53,5 +44,5 @@
             <inertial>
             <!--assign inertial properties to drive wheels -->
-            <mass value="1" />
+            <mass value="${1*default_mass}" />
             <inertia ixx="0.1" ixy="0" ixz="0"
               iyy="0.1" iyz="0"
@@ -82,5 +73,5 @@
             <inertial>
             <!--assign inertial properties to drive wheels -->
-            <mass value="1.5" />
+            <mass value="${0.1*default_mass}" />
             <inertia ixx="0.1" ixy="0" ixz="0"
               iyy="0.1" iyz="0"
@@ -109,6 +100,5 @@
         </collision>
         <inertial>
-            <!--assign almost all the mass to the main body box; set m= 100kg; treat I as approx m*r^2 -->
-            <mass value="100" />
+            <mass value="${0.1*default_mass}" />
             <inertia ixx="10" ixy="0" ixz="0"
               iyy="10" iyz="0"
@@ -136,5 +126,5 @@
         <inertial>
             <!--assign almost all the mass to the main body box; set m= 100kg; treat I as approx m*r^2 -->
-            <mass value="50" />
+            <mass value="${1.0*default_mass}" />
             <inertia ixx="10" ixy="0" ixz="0"
               iyy="10" iyz="0"
@@ -159,5 +149,5 @@
       </visual>
       <inertial>
-          <mass value="4.0" />
+          <mass value="${0.1*default_mass}" />
           <inertia ixx="0.01" ixy="0" ixz="0" iyy="0.01" iyz="0" izz="0.01" />
       </inertial>
@@ -245,4 +235,5 @@
         <xacro:wheel_controller_plugin wheelset1="2" wheelset2="2"/>
     </gazebo>
+<!--
     <xacro:macro name="friction_macro" params="wheelnum constant">
         <gazebo reference="left${wheelnum}_wheel">
@@ -262,4 +253,22 @@
     <xacro:friction_macro wheelnum="3" constant="100000.0"/>
     <xacro:friction_macro wheelnum="4" constant="100000.0"/>
+  -->
+    <xacro:macro name="friction_macro" params="wheelnum mu1 mu2">
+        <gazebo reference="left${wheelnum}_wheel">
+            <mu1>${mu1}</mu1>
+            <mu2>${mu2}</mu2>
+            <material >Gazebo/Black </material >
+        </gazebo>
+        <gazebo reference="right${wheelnum}_wheel">
+            <mu1>${mu1}</mu1>
+            <mu2>${mu2}</mu2>
+            <material >Gazebo/Black </material >
+        </gazebo>
+    </xacro:macro>
+    <xacro:friction_macro wheelnum="0" mu1="200.0" mu2="100.0"/>
+    <xacro:friction_macro wheelnum="1" mu1="200.0" mu2="100.0"/>
+    <xacro:friction_macro wheelnum="2" mu1="200.0" mu2="100.0"/>
+    <xacro:friction_macro wheelnum="3" mu1="200.0" mu2="100.0"/>
+    <xacro:friction_macro wheelnum="4" mu1="200.0" mu2="100.0"/>
     <gazebo reference="base_link">
         <material >Gazebo/Orange </material >

Commit message: minor changes

File: packages/sentry/sentry_urdf/urdf/sentry.xacro (robot description, xacro)
@@ -235,23 +235,4 @@
         <xacro:wheel_controller_plugin wheelset1="2" wheelset2="2"/>
     </gazebo>
-<!--
-    <xacro:macro name="friction_macro" params="wheelnum constant">
-        <gazebo reference="left${wheelnum}_wheel">
-            <mu1>${constant}</mu1>
-            <mu2>${constant}</mu2>
-            <material >Gazebo/Black </material >
-        </gazebo>
-        <gazebo reference="right${wheelnum}_wheel">
-            <mu1>${constant}</mu1>
-            <mu2>${constant}</mu2>
-            <material >Gazebo/Black </material >
-        </gazebo>
-    </xacro:macro>
-    <xacro:friction_macro wheelnum="0" constant="100000.0"/>
-    <xacro:friction_macro wheelnum="1" constant="100000.0"/>
-    <xacro:friction_macro wheelnum="2" constant="100000.0"/>
-    <xacro:friction_macro wheelnum="3" constant="100000.0"/>
-    <xacro:friction_macro wheelnum="4" constant="100000.0"/>
-  -->
     <xacro:macro name="friction_macro" params="wheelnum mu1 mu2">
         <gazebo reference="left${wheelnum}_wheel">

Commit message: created transforms for robot, renamed stuff to match hardware other stuff

File: packages/sentry/sentry_urdf/urdf/sentry.xacro (robot description, xacro)
@@ -52,5 +52,5 @@
         <joint name="${prefix}_wheel_joint" type="continuous">
             <axis xyz="0 0 1"/>
-            <parent link="base_link"/>
+            <parent link="base_laser1_link"/>
             <child link="${prefix}_wheel"/>
             <origin xyz="${displacement} ${left*track/2} ${-bodyheight/2 + zDisp}" rpy="0 ${M_PI/2} ${M_PI/2}"/>
@@ -81,5 +81,5 @@
         <joint name="${prefix}_big_wheel_joint" type="continuous">
             <axis xyz="0 0 1"/>
-            <parent link="base_link"/>
+            <parent link="base_laser1_link"/>
             <child link="${prefix}_big_wheel"/>
             <origin xyz="${displacement} ${left*track/2} ${bigtirerad + zDisp}" rpy="0 ${M_PI/2} ${M_PI/2}"/>
@@ -107,9 +107,9 @@
     </link>
     <joint name="masttobase" type="fixed">
-        <parent link="base_link"/>
+        <parent link="base_laser1_link"/>
         <child link="mast"/>
         <origin xyz="${bodylen/4} 0 ${mastheight/2 + bodyheight/2 + zDisp}" rpy="0 0 0"/>
     </joint>
-    <link name="base_link">
+    <link name="base_laser1_link">
         <visual>
             <geometry>
@@ -157,5 +157,5 @@
       <axis xyz="0 1 0" />
       <origin xyz="${bodylen/2 + lidar_cube_size/2} 0 ${lidar_cube_size/2 - bodyheight/2 + zDisp}" rpy="0 0 0"/>
-      <parent link="base_link"/>
+      <parent link="base_laser1_link"/>
       <child link="lidar_link"/>
   </joint>
@@ -218,5 +218,5 @@
         <wheelSeparation>${track}</wheelSeparation>
         <wheelDiameter>${tirediam}</wheelDiameter>
-        <robotBaseFrame>base_link</robotBaseFrame>
+        <robotBaseFrame>base_laser1_link</robotBaseFrame>
         <torque>200</torque>
         <topicName>cmd_vel</topicName>
@@ -252,5 +252,5 @@
     <xacro:friction_macro wheelnum="3" mu1="200.0" mu2="100.0"/>
     <xacro:friction_macro wheelnum="4" mu1="200.0" mu2="100.0"/>
-    <gazebo reference="base_link">
+    <gazebo reference="base_laser1_link">
         <material >Gazebo/Orange </material >
     </gazebo>

Commit message: created some transforms, renamed some stuff

File: packages/sentry/sentry_urdf/urdf/sentry.xacro (robot description, xacro)
@@ -52,5 +52,5 @@
         <joint name="${prefix}_wheel_joint" type="continuous">
             <axis xyz="0 0 1"/>
-            <parent link="base_laser1_link"/>
+            <parent link="base_link"/>
             <child link="${prefix}_wheel"/>
             <origin xyz="${displacement} ${left*track/2} ${-bodyheight/2 + zDisp}" rpy="0 ${M_PI/2} ${M_PI/2}"/>
@@ -81,5 +81,5 @@
         <joint name="${prefix}_big_wheel_joint" type="continuous">
             <axis xyz="0 0 1"/>
-            <parent link="base_laser1_link"/>
+            <parent link="base_link"/>
             <child link="${prefix}_big_wheel"/>
             <origin xyz="${displacement} ${left*track/2} ${bigtirerad + zDisp}" rpy="0 ${M_PI/2} ${M_PI/2}"/>
@@ -107,9 +107,9 @@
     </link>
     <joint name="masttobase" type="fixed">
-        <parent link="base_laser1_link"/>
+        <parent link="base_link"/>
         <child link="mast"/>
         <origin xyz="${bodylen/4} 0 ${mastheight/2 + bodyheight/2 + zDisp}" rpy="0 0 0"/>
     </joint>
-    <link name="base_laser1_link">
+    <link name="base_link">
         <visual>
             <geometry>
@@ -157,5 +157,5 @@
       <axis xyz="0 1 0" />
       <origin xyz="${bodylen/2 + lidar_cube_size/2} 0 ${lidar_cube_size/2 - bodyheight/2 + zDisp}" rpy="0 0 0"/>
-      <parent link="base_laser1_link"/>
+      <parent link="base_link"/>
       <child link="lidar_link"/>
   </joint>
@@ -218,5 +218,5 @@
         <wheelSeparation>${track}</wheelSeparation>
         <wheelDiameter>${tirediam}</wheelDiameter>
-        <robotBaseFrame>base_laser1_link</robotBaseFrame>
+        <robotBaseFrame>base_link</robotBaseFrame>
         <torque>200</torque>
         <topicName>cmd_vel</topicName>
@@ -252,5 +252,5 @@
     <xacro:friction_macro wheelnum="3" mu1="200.0" mu2="100.0"/>
     <xacro:friction_macro wheelnum="4" mu1="200.0" mu2="100.0"/>
-    <gazebo reference="base_laser1_link">
+    <gazebo reference="base_link">
         <material >Gazebo/Orange </material >
     </gazebo>
